File: Hardware/PowerBoard.sch (EAGLE design)
At the start: 71 parts, among them IC1 68008, IC11 NE555, IC12 74HC08N, IC13 74HC05, IC2 AS6C1008, IC3 39SF020, IC4 DS1244Y, IC5 68681, IC6 74HC30N, IC7 74HC04N, IC8 74HC138N, IC9 74HC7266, Q1 3.6864MHz

Commit message: revamped power connections; moved power regulation to separate board (plus RS232 conversion)
Parts:
- removed C11, C15, C16, C17, C18, C19, C20, C21, C28, C9: 100nF, rcl:C-EUC0805
- removed C14: 10µF, rcl:CPOL-EUSMCB
- removed IC11: NE555, st-microelectronics:NE555
- removed IC12: 74HC08N, 74xx-eu:74HC08N
- removed IC13: 74HC05, 74xx-eu:74HCT05N
- removed IC3: 39SF020, Parts:SST39SF0X0PDIP32
- removed IC4: DS1244Y, Parts:DS1244EDIP-28
- removed IC5: 68681, Parts:MC68681PLCC44-SOCKET
- removed IC6: 74HC30N, 74xx-eu:74HC30N
- removed IC7: 74HC04N, 74xx-eu:74HC04N
- removed IC8: 74HC138N, 74xx-eu:74HC138N
- removed IC9: 74HC7266, 74xx-eu:74HC266N
- removed LED2, LED3, LED4, LED6: (no value), led:LEDCHIPLED_1206
- removed Q1: 3.6864MHz, crystal:XO-8
- removed R10, R11, R12, R14, R15, R17, R4, R5, R6, R9: 10k, rcl:R-EU_R2012
- removed R16, R18: 1M, rcl:R-EU_R2012
- removed R19, R2, R20, R21, R3, R7, R8: 3k, rcl:R-EU_R2012
- removed WEED1: WEED, Parts:WEED
- added C26: 100nF, rcl:C-EUC0805
- added H1, H2, H3: MOUNT-HOLE2.8, holes:MOUNT-HOLE2.8
- added SV7: 1792863, Parts:1792863
- added X1, X2: (no value), con-subd:F09HPS
- C1, C2, C5, C6: value 100nF -> 2.2µF; MOUSER 710-885012207072 -> 710-885012107016
- C10, C8: value 10µF -> 1µF; device rcl:CPOL-EUSMCB -> rcl:C-EUC0805; MOUSER 581-TAJB106K020RNJV -> 710-885012107015
- C12, C13: value 100nF -> 1µF; MOUSER 710-885012207072 -> 710-885012107015
- IC1: value 68008 -> MAX232; device Parts:MC68008P -> maxim:MAX232; MOUSER (none) -> 595-MAX232N
- IC2: value AS6C1008 -> 7805; device Parts:AS6C1008 -> linear:7805TV; MOUSER (none) -> 490-VXO7805-1000
- LED1: MOUSER 710-156120RS75300 -> 710-156120YS75300
- S2: device switch-omron:10-XX -> switch-dil:DP04; MOUSER 653-B3F-1052 -> 611-BDB04
- SV1: device con-lstb:MA10-2 -> con-lstb:MA04-2
- SV2: device con-lstb:MA07-2 -> con-lstb:MA03-2
- SV6: device con-lstb:MA05-2 -> con-lstb:MA04-2
Connections:
- removed net !68681_CS: IC5.!CS, IC8A.Y2
- removed net !68681_DTACK: IC5.!DTACK, IC6A.I7, R1.1
- removed net !68681_IACK: IC5.!IACK, IC7C.O
- removed net !AS: IC1.AS, IC8A.G2B
- removed net !BG: IC1.BG
- removed net !DS: IC1.DS
- removed net !DTACK: IC1.DTACK, IC7A.O, LED6.C
- removed net !HALT: IC1.HALT, IC13B.O, LED2.C, R17.1
- removed net !IPL1: IC1.IPL1, IC5.!INTR
- removed net !NIXIE_CS: IC6A.I5, IC8A.Y4, SV1.17
- removed net !OE: IC2.!OE, IC3.!OE, IC4.!OE, IC7B.O
- removed net !RAM_CS: IC2.!CE1, IC6A.I3, IC9B.O, R3.1
- removed net !RAM_CS0: IC8A.Y6, IC9B.I1
- removed net !RAM_CS1: IC8A.Y7, IC9B.I0
- removed net !RESET: IC1.RESET, IC13A.O, IC5.!RESET, LED1.C, R4.1
- removed net !ROM_CS: IC3.!CS, IC6A.I2, IC9A.O, R2.1
- removed net !ROM_CS0: IC8A.Y0, IC9A.I0
- removed net !ROM_CS1: IC8A.Y1, IC9A.I1
- removed net !RTC_CS: IC4.!CS, IC6A.I4, IC8A.Y3
- removed net !VFD_CS: IC6A.I6, IC8A.Y5, SV2.5
- removed net !VFD_RESET: IC5.OP4, SV2.4
- removed net A0: IC1.A0, IC2.A0, IC3.A0, IC4.A0, IC5.A1, SV1.3
- removed net A1: IC1.A1, IC2.A1, IC3.A1, IC4.A1, IC5.A2, SV1.5
- removed net A10: IC1.A10, IC2.A10, IC3.A10, IC4.A10
- removed net A11: IC1.A11, IC2.A11, IC3.A11, IC4.A11
- removed net A12: IC1.A12, IC2.A12, IC3.A12, IC4.A12
- removed net A13: IC1.A13, IC2.A13, IC3.A13, IC4.A13
- removed net A14: IC1.A14, IC2.A14, IC3.A14, IC4.A14
- removed net A15: IC1.A15, IC2.A15, IC3.A15
- removed net A16: IC1.A16, IC2.A16, IC3.A16, IC8A.A
- removed net A17: IC1.A17, IC8A.B
- removed net A18: IC1.A18, IC8A.C
- removed net A19: IC1.A19
- removed net A2: IC1.A2, IC2.A2, IC3.A2, IC4.A2, IC5.A3, SV1.7
- removed net A3: IC1.A3, IC2.A3, IC3.A3, IC4.A3, IC5.A4, SV1.9
- removed net A4: IC1.A4, IC2.A4, IC3.A4, IC4.A4, SV1.11
- removed net A5: IC1.A5, IC2.A5, IC3.A5, IC4.A5
- removed net A6: IC1.A6, IC2.A6, IC3.A6, IC4.A6
- removed net A7: IC1.A7, IC2.A7, IC3.A7, IC4.A7
- removed net A8: IC1.A8, IC2.A8, IC3.A8, IC4.A8
- removed net A9: IC1.A9, IC2.A9, IC3.A9, IC4.A9
- removed net CLK: IC1.CLK, IC5.X1/CLK, Q1.OUT
- removed net D0: IC1.D0, IC2.D0, IC3.DQ0, IC4.DQ0, IC5.D0, R5.2, SV1.8, SV2.7
- removed net D1: IC1.D1, IC2.D1, IC3.DQ1, IC4.DQ1, IC5.D1, R6.2, SV1.6, SV2.8
- removed net D2: IC1.D2, IC2.D2, IC3.DQ2, IC4.DQ2, IC5.D2, R9.2, SV1.4, SV2.9
- removed net D3: IC1.D3, IC2.D3, IC3.DQ3, IC4.DQ3, IC5.D3, R10.2, SV1.10, SV2.10
- removed net D4: IC1.D4, IC2.D4, IC3.DQ4, IC4.DQ4, IC5.D4, R11.2, SV1.12, SV2.11
- removed net D5: IC1.D5, IC2.D5, IC3.DQ5, IC4.DQ5, IC5.D5, R12.2, SV1.14, SV2.12
- removed net D6: IC1.D6, IC2.D6, IC3.DQ6, IC4.DQ6, IC5.D6, R14.2, SV1.16, SV2.13
- removed net D7: IC1.D7, IC2.D7, IC3.DQ7, IC4.DQ7, IC5.D7, R15.2, SV1.18, SV2.14
- removed net E: IC1.E
- removed net FC0: IC1.FC0, IC12A.I0
- removed net FC1: IC1.FC1, IC12B.I0
- removed net FC2: IC1.FC2, IC12B.I1
- removed net N$7 (its old number): LED3.A, R7.2
- removed net OUT0: IC5.OP3, SV6.8
- removed net OUT1: IC5.OP1, SV6.7
- removed net R/!W!: IC1.R/!W, IC2.!WE, IC3.!WE, IC4.!WE, IC5.R/!W, IC7B.I, SV1.13
- removed net RESET: IC11.OUT, IC13A.I, IC13B.I
- removed net STATUS0: IC5.OP7, R8.1
- removed net STATUS1: IC5.OP5, R7.1
- removed net SW0: IC5.IP1, SV6.1
- removed net SW1: IC5.IP0, SV6.2
- removed net SW2: IC5.IP2, SV6.3
- removed net VFD_BUSY: IC5.IP3, SV2.3
- new net +12V: C12.1, C26.1, IC2.VI, R1.1, SV1.3, SV1.5, SV1.7, SV7.2
- new net N$13: IC1G$1.T1IN, S2.8
- new net N$4: C5.1, IC1G$1.C1+
- new net N$8: LED1.A, R1.2
- new net SER0_IN: IC1G$1.R1IN, X1-3.F
- new net SER0_OUT: IC1G$1.T1OUT, X1-2.F
- new net SER1_IN: IC1G$1.R2IN, X2-3.F
- new net SER1_OUT: IC1G$1.T2OUT, X2-2.F
- net +5V: now also C10.1, C8.1, IC1P.VCC, IC2.VO, SV1.1, SV2.1, SV2.3, SV2.5, SV6.8; no longer C1.1, C10.+, C11.1, C12.1, C14.+, C15.1, C16.1, C17.1, C2.1, C20.1, C21.1, C28.1, C5.1, C6.1, C8.+, C9.1, IC1.BERR, IC1.BR, IC1.VCC, IC1.VPA, IC11./RES, IC11.VCC+, IC12P.VCC, IC13P.VCC, IC2.CE2, IC2.VCC, IC3.VCC, IC4.VCC, IC5.VCC, IC6A.I0, IC6A.I1, IC6P.VCC, IC7P.VCC, IC8A.G1, IC8P.VCC, IC9P.VCC, Q1.VCC, R1.2, R16.1, R17.2, R18.1, R19.1, R2.2, R20.1, R21.1, R3.2, R4.2, SV1.19, SV2.2, SV5.6, SV5.8
- net GND: now also C10.2, C26.2, C8.2, IC1P.GND, LED1.C, SV1.4, SV1.6, SV1.8, SV2.2, SV2.4, SV2.6, SV6.7, SV7.1, X1-5.F, X1-G.G1, X2-5.F, X2-G.G1; no longer C10.-, C11.2, C14.-, C15.2, C16.2, C17.2, C18.2, C19.2, C20.2, C21.2, C28.2, C5.2, C6.2, C8.-, C9.2, IC1.GND@1, IC1.GND@2, IC1.IPL0/2, IC11.CON, IC11.GND, IC12C.I0, IC12C.I1, IC12D.I0, IC12D.I1, IC12P.GND, IC13C.I, IC13D.I, IC13E.I, IC13F.I, IC13P.GND, IC3.A17, IC3.A18, IC3.GND, IC4.GND, IC5.GND, IC6P.GND, IC7D.I, IC7E.I, IC7F.I, IC7P.GND, IC8A.G2A, IC8P.GND, IC9C.I0, IC9C.I1, IC9D.I0, IC9D.I1, IC9P.GND, LED3.C, LED4.C, Q1.GND, R10.1, R11.1, R12.1, R14.1, R15.1, R5.1, R6.1, R9.1, S2.P, S2.P1, SV1.1, SV1.20, SV2.1
- net N$1: now also C1.1, IC1G$1.V+; no longer C18.1, IC11.TRI, R16.2, S2.S, S2.S1
- net N$10: now also C5.2, IC1G$1.C1-; no longer LED6.A, R21.2
- net N$11: now also IC1G$1.R1OUT, S2.6; no longer IC12A.I1, IC12B.O
- net N$12: now also IC1G$1.T2IN, S2.7; no longer C19.1, IC11.DIS, IC11.TRE, R18.2
- net N$2: now also C2.1, IC1G$1.V-; no longer LED1.A, R19.2
- net N$3: now also C6.1, IC1G$1.C2+; no longer IC6A.O, IC7A.I
- net N$5: now also SV5.6, SV5.8; no longer IC12A.O, IC7C.I
- net N$6: now also IC1G$1.R2OUT, S2.5; no longer LED2.A, R20.2
- net N$9: now also C6.2, IC1G$1.C2-; no longer LED4.A, R8.2
- net UART0_RX: now also S2.3, SV6.4; no longer IC5.RXDA
- net UART0_TX: now also S2.1, SV6.3; no longer IC5.TXDA
- net UART1_RX: now also S2.4, SV6.2; no longer IC5.RXDB
- net UART1_TX: now also S2.2, SV6.1; no longer IC5.TXDB
Other:
- note added: "SV1: To HV supply SV2-4: Regulated 5V"
- note added: "SV5: UART from CPU board SV4: UART at TTL level"
- note added: "SV5: UART from CPU board SV6: UART at TTL level Use DIP switch S1 to select which UARTs are TTL or RS232 level"
- note added: "X1: UART0 RS232 X2: UART1 RS232"
- note removed: "!CS! generator (see memory map)"
- note removed: "!DTACK! generator"
- note removed: "!IACK! generator for 68681"
- note removed: "!OE! generator (= !R/!W!)"
- note removed: "!RESET! generator"
- note removed: "$40000 - $4FFFF: Nixie output registers $50000 - $5FFFF: VFD $60000 - $7FFFF: RAM"
- note removed: "1x 100nF per 74xxx IC"
- note removed: "1x 10µF for VFD/Nixie connector 1x 100nF for each IC and connector"
- note removed: "1x 10µF for each 68008 and RAM/ROM 1x 100nF for each IC and oscillator 1x 100nF for PoR monitor"
- note removed: "IC10 can be substituted for any 7805 compatible with > 1A current"
- note removed: "Memory Map: $00000 - $1FFFF: ROM $20000 - $2FFFF: 68681 $30000 - $3FFFF: RTC"
- note removed: "R2/R3 may not be needed, populate if RAM/ROM !CS! is bad"
- note removed: "S1: reset switch"
- note removed: "SV1: Nixie Board SV2: VFD (Noritake CU24043-Y100) SV6: Side buttons"
- note removed: "SV5: UARTs"
- note removed: "Unused gates"

Commit message: Added HV supply; cleaned up power board
Parts:
- renumbered C1 to C104, C10 to C207, C12 to C202, C13 to C206, C2 to C103, C24 to C203, C25 to C204, C26 to C201, C3 to C105, C4 to C107, C5 to C101, C6 to C102, C7 to C106, C8 to C205, H1 to H101, H2 to H102, H3 to H103, IC1 to IC101, IC2 to IC201, LED1 to LED201, LED5 to LED202, R1 to R201, R13 to R202, S2 to S101, SV1 to SV202, SV2 to SV203, SV3 to SV204, SV5 to SV101, SV6 to SV102, SV7 to SV201, X1 to X101, X2 to X102
Other:
- note added: "SV101: UART from CPU board SV102: UART at TTL level Use DIP switch S101 to select which UARTs are TTL or RS232 level"
- note added: "SV201: +12VDC input SV202: To HV supply SV203-204: Regulated 5V"
- note added: "X101: UART0 RS232 X102: UART1 RS232"
- note removed: "SV1: To HV supply SV2-4: Regulated 5V"
- note removed: "SV5: UART from CPU board SV4: UART at TTL level"
- note removed: "SV5: UART from CPU board SV6: UART at TTL level Use DIP switch S1 to select which UARTs are TTL or RS232 level"
- note removed: "X1: UART0 RS232 X2: UART1 RS232"
