File: Hardware/TubeBoard-Logic.sch (EAGLE design)
At the start: 33 parts, among them IC1 74HC573D, IC2 74HC573D, IC3 74HC85D, IC4 74HC08D, IC5 74HC04D, IC6 MKE04Z8, IC7 74HC139D, IC8 74HC573D, J1 CORTEX_DEBUG_PTH

Commit message: finished routing basic data latch only tube logic board
Parts:
- removed C7: 100nF, rcl:C-EUC1206
- removed C8: 10µF, rcl:CPOL-EUSMCB
- removed IC6: MKE04Z8, Parts:MKE04Z8SOIC20
- removed IC8: 74HC573D, 74xx-eu:74HC573D
- removed J1: CORTEX_DEBUG_PTH, SparkFun-Connectors:CORTEX_DEBUG_PTH
- removed LED1: (no value), led:LEDCHIPLED_1206
- removed R4: 3k, rcl:R-EU_R2012
- removed SV4: (no value), con-lstb:MA03-1
Connections:
- removed net !ARM_RESET: IC6.PA5, J1.!RESET
- removed net !PWM_LATCH: IC5D.I, IC7A.Y2
- removed net ARM_SWDCLK: IC6.PA0/SWDCLK, J1.SWDCLK/TCK
- removed net ARM_SWDIO: IC6.PA4/SWDIO, J1.SWDIO/TMS
- removed net N$9: LED1.A, R4.2
- removed net PWM_D0: IC6.PB7, IC8A.1Q
- removed net PWM_D1: IC6.PB6, IC8A.2Q
- removed net PWM_D2: IC6.PB5, IC8A.3Q
- removed net PWM_D3: IC6.PB4, IC8A.4Q
- removed net PWM_LATCH: IC5D.O, IC6.PB3, IC8A.OC
- removed net STATUS0: IC6.PA3, R4.1
- removed net UART_RX: IC6.PB0, SV4.2
- removed net UART_TX: IC6.PB1, SV4.3
- net +5V: no longer C7.1, C8.+, IC6.VDD, IC8P.VCC, J1.VCC
- net D0: no longer IC8A.1D
- net D1: no longer IC8A.2D
- net D2: no longer IC8A.3D
- net D3: no longer IC8A.4D
- net D4: no longer IC8A.5D
- net D5: no longer IC8A.6D
- net D6: no longer IC8A.7D
- net D7: no longer IC8A.8D
- net GND: now also IC5D.I; no longer C7.2, C8.-, IC6.GND, IC8A.C, IC8P.GND, J1.GND@3, J1.GND@5, J1.GNDDTCT, LED1.C, SV4.1
- net PWM0: now also IC2A.5Q; no longer IC6.PC0
- net PWM1: now also IC2A.6Q; no longer IC6.PC1
- net PWM2: now also IC2A.7Q; no longer IC6.PC2
- net PWM3: now also IC2A.8Q; no longer IC6.PC3
